File: E10.kicad_pcb (KiCad board)
At the start: 2 copper layers, 59.9 x 21.6 mm, 45 parts, among them J1 Conn_01x17_Male, J2 Conn_01x03_Male, J3 Conn_01x03_Male, J4 Conn_01x06_Male, J5 Conn_01x06_Male, J6 Conn_01x17_Male, J7 Conn_01x17_Male, U1 AVR-64da32, U2 MIC5205-3.3YM5

Commit message: Initial commit
Other:
- board text removed: "Svo-PWR"

Commit message: Initial commit
Parts:
- C1: value 4.7u -> 22u
- C5: value 47u -> 22u
- J2: value Conn_01x03_Male -> WS-bus output
- J3: value Conn_01x03_Male -> WS-bus input
- J4: value Conn_01x06_Male -> UPDI
- J5: value Conn_01x06_Male -> Debug
- JP3: value Jumper_3_Open -> LED common
- R1: value 6.8k -> 3.3k
- R10, R11, R12, R13, R14, R15, R17, R2, R3, R4, R5, R6, R7, R8, R9: value 160 -> 220
- R16: value 4.7k -> 220
- R20: value 2.2k -> 3.3k
- R23: value 160 -> 27
- moved J2 1.36 mm to (147.8, 88.8)
- moved J3 1.17 mm to (94.0, 88.9)
- moved JP3 0.58 mm to (98.1, 79.3)
Connections:
- J7 pad 9: (no net) -> GND
Routing:
- net +5V: track 82.7 -> 91.3 mm
- net Net-(R18-Pad1): track 33.6 -> 34.8 mm
Other:
- board text added: "Hbt"
- board text removed: "MSG"

Commit message: Initial commit
Parts:
- removed C5: 22u, Capacitor_SMD:C_1206_3216Metric
- removed D4: ERR(red), LED_SMD:LED_0603_1608Metric
- removed J6: Conn_01x17_Male, WSnOUT:PinHeader_1x17_P2.54mm_Vertical_NoCrtYd
- removed JP2: Jumper_3_Open, Jumper:SolderJumper-3_P1.3mm_Open_RoundedPad1.0x1.5mm
- removed JP3: LED common, Jumper:SolderJumper-3_P1.3mm_Open_RoundedPad1.0x1.5mm
- removed R1: 3.3k, Resistor_SMD:R_0603_1608Metric
- removed R22, R24: t.b.d., Resistor_SMD:R_0603_1608Metric
- removed R23: 27, Resistor_SMD:R_0603_1608Metric
- removed U2: MIC5205-3.3YM5, Package_TO_SOT_SMD:SOT-23-5
- C1: value 22u -> 1u; moved to B.Cu
- J1, J7: value Conn_01x17_Male -> Conn_01x09; footprint WSnOUT:PinHeader_1x17_P2.54mm_Vertical_NoCrtYd -> RTB_parts:1725724
- moved C1 25.9 mm to (120.9, 81.0), turned to 0 degrees
- moved J7 21.9 mm to (122.2, 78.4), turned to 0 degrees
- moved J4 2.97 mm to (128.3, 95.4), turned to 90 degrees
- moved D2 1.55 mm to (120.9, 95.8)
- moved R20 1.55 mm to (120.9, 95.8)
- moved J1 1.52 mm to (99.3, 78.4), turned to 0 degrees
Connections:
- C2 pad 1: VDD -> +5V
- C3 pad 1: VDD -> +5V
- J1 pad 1: Net-(J1-Pad1) -> OUT0
- J1 pad 2: Net-(J1-Pad1) -> OUT1
- J1 pad 3: Net-(J1-Pad1) -> OUT2
- J1 pad 4: Net-(J1-Pad1) -> OUT3
- J1 pad 5: Net-(J1-Pad1) -> OUT4
- J1 pad 6: Net-(J1-Pad1) -> OUT5
- J1 pad 7: Net-(J1-Pad1) -> OUT6
- J1 pad 8: Net-(J1-Pad1) -> OUT7
- J1 pad 9: Net-(J1-Pad1) -> +5V
- J4 pad 2: VDD -> +5V
- J5 pad 3: VDD -> +5V
- J7 pad 1: OUT0 -> GND
- J7 pad 2: OUT1 -> OUT8
- J7 pad 3: OUT2 -> OUT9
- J7 pad 4: OUT3 -> OUT10
- J7 pad 5: OUT4 -> OUT11
- J7 pad 6: OUT5 -> OUT12
- J7 pad 7: OUT6 -> OUT13
- J7 pad 8: OUT7 -> OUT14
- J7 pad 9: GND -> OUT15
- R20 pad 2: VDD -> +5V
- U1 pad 16: Net-(R23-Pad1) -> Net-(R5-Pad1)
- U1 pad 17: Net-(R5-Pad1) -> (no net)
- U1 pad 18: VDD -> +5V
- U1 pad 25: Net-(D4-Pad1) -> (no net)
- U1 pad 26: Net-(R22-Pad1) -> (no net)
- U1 pad 28: VDD -> +5V
Routing:
- net +5V: track 91.3 -> 19.1 mm
- net Net-(J1-Pad1): track 43.7 -> 0.00 mm
- net Net-(R23-Pad1): track 20.6 -> 0.00 mm, vias 1 -> 0
- net VDD: track 17.1 -> 0.00 mm, vias 4 -> 0
- net Net-(R19-Pad1): track 37.6 -> 27.4 mm
- net Net-(R18-Pad1): track 34.8 -> 26.8 mm
- net Net-(R22-Pad1): track 5.14 -> 0.00 mm, vias 1 -> 0
- net +3V3: track 4.38 -> 0.00 mm
- net DAC: track 4.28 -> 0.00 mm
- net OUT9: track 3.00 -> 6.87 mm
- net OUT15: track 3.02 -> 6.90 mm
- net OUT14: track 3.02 -> 6.90 mm
- net OUT11: track 3.02 -> 6.90 mm
- net OUT10: track 3.02 -> 6.90 mm
- net OUT8: track 3.02 -> 6.90 mm
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- added copper zone on F.Cu, net +5V
- removed copper zone on F.Cu, net VDD
Other:
- rule solder_mask_min_width: 0.25 -> 0.1
- board text added: "+|-"
- board text added: "1"
- board text added: "16"
- board text added: "8"
- board text added: "9"
- board text added: "[Debug IF]"
- board text removed: "+"
- board text removed: "5V|3V"
- board text removed: "P/E"
- board text removed: "PWM"
- board text removed: "[Code]"
- board text removed: "[V24,1Mb,8N1,RTS]"

Commit message: Initial commit
Parts:
- added C4: 4.7u/10V, Capacitor_SMD:C_0805_2012Metric, F.Cu at (155.9, 94.5)
- added D1: SS34F, Diode_SMD:D_SOD-123F, B.Cu at (164.3, 87.7)
- added J6: LED common, RTB_parts:1725656, F.Cu at (158.2, 78.6)
- added J8: LED 16-17, RTB_parts:1725656, F.Cu at (102.6, 78.6)
- added JP1: SolderJumper_2_Open, Jumper:SolderJumper-2_P1.3mm_Open_RoundedPad1.0x1.5mm, F.Cu at (158.7, 91.2)
- added JP2: SolderJumper_3_Open, Jumper:SolderJumper-3_P1.3mm_Open_RoundedPad1.0x1.5mm, B.Cu at (159.5, 81.5)
- added R21: 220, Resistor_SMD:R_0603_1608Metric, F.Cu at (105.1, 85.6)
- added R22: 220, Resistor_SMD:R_0603_1608Metric, F.Cu at (102.5, 85.5)
- added R23: 22, Resistor_SMD:R_0603_1608Metric, B.Cu at (155.7, 84.7)
- added R24: 47k, Resistor_SMD:R_0603_1608Metric, F.Cu at (155.0, 85.5)
- added U2: MIC5205-5.0YM5, Package_TO_SOT_SMD:SOT-23-5, F.Cu at (158.7, 94.3)
- added U3: MCP6001, Package_TO_SOT_SMD:SOT-23-5, F.Cu at (157.5, 85.6)
- C1: value 1u -> 4.7u/10V; footprint Capacitor_SMD:C_1206_3216Metric -> Capacitor_SMD:C_0805_2012Metric; moved to F.Cu
- C2, C3: value 1u -> 100n
- J1: value Conn_01x09 -> LED 8-15; footprint RTB_parts:1725724 -> RTB_parts:1725711
- J7: value Conn_01x09 -> LED 0-7; footprint RTB_parts:1725724 -> RTB_parts:1725711
- R20: value 3.3k -> 4.7k
- R25: value t.b.d. -> 47k; moved to F.Cu
- moved J3 73.3 mm to (167.2, 88.9)
- moved R18 64.1 mm to (162.2, 85.6), turned to 90 degrees
- moved J2 53.8 mm to (94.0, 89.0)
- moved R25 53.3 mm to (153.5, 85.5), turned to 90 degrees
- moved R19 44.0 mm to (99.8, 85.6), turned to 90 degrees
- moved C1 42.8 mm to (161.5, 94.5), turned to 90 degrees
- moved J1 19.9 mm to (119.2, 78.6)
- moved J7 19.8 mm to (142.1, 78.6)
- moved H3 19.4 mm to (167.3, 78.4)
- moved H4 19.4 mm to (167.2, 94.0)
- moved C2 10.1 mm to (126.2, 91.5)
- moved J4 9.71 mm to (138.0, 95.4)
- moved R10 9.71 mm to (140.8, 85.6)
- moved R11 9.71 mm to (138.2, 85.6)
- moved R14 9.71 mm to (150.9, 85.6)
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Connections:
- C2 pad 1: +5V -> VDD
- C3 pad 1: +5V -> VDD
- J1 pad 1: OUT0 -> OUT15
- J1 pad 2: OUT1 -> OUT14
- J1 pad 3: OUT2 -> OUT13
- J1 pad 4: OUT3 -> OUT12
- J1 pad 5: OUT4 -> OUT11
- J1 pad 6: OUT5 -> OUT10
- J1 pad 7: OUT6 -> OUT9
- J1 pad 8: OUT7 -> OUT8
- J4 pad 2: +5V -> VDD
- J5 pad 3: +5V -> VDD
- J7 pad 1: GND -> OUT7
- J7 pad 2: OUT8 -> OUT6
- J7 pad 3: OUT9 -> OUT5
- J7 pad 4: OUT10 -> OUT4
- J7 pad 5: OUT11 -> OUT3
- J7 pad 6: OUT12 -> OUT2
- J7 pad 7: OUT13 -> OUT1
- J7 pad 8: OUT14 -> OUT0
- R10 pad 2: OUT11 -> OUT4
- R11 pad 2: OUT10 -> OUT5
- R12 pad 2: OUT9 -> OUT6
- R13 pad 2: OUT8 -> OUT7
- R14 pad 2: OUT15 -> OUT0
- R15 pad 2: OUT14 -> OUT1
- R16 pad 2: OUT13 -> OUT2
- R17 pad 2: OUT12 -> OUT3
- R2 pad 2: OUT3 -> OUT12
- R20 pad 2: +5V -> VDD
- R25 pad 1: GND -> Net-(R24-Pad1)
- R25 pad 2: V24.cts -> GND
- R3 pad 2: OUT2 -> OUT13
- R4 pad 2: OUT1 -> OUT14
- R5 pad 2: OUT0 -> OUT15
- R6 pad 2: OUT7 -> OUT8
- R7 pad 2: OUT6 -> OUT9
- R8 pad 2: OUT5 -> OUT10
- R9 pad 2: OUT4 -> OUT11
- U1 pad 16: Net-(R5-Pad1) -> DAC
- U1 pad 17: (no net) -> Net-(R5-Pad1)
- U1 pad 18: +5V -> VDD
- U1 pad 25: (no net) -> Net-(R22-Pad1)
- U1 pad 28: +5V -> VDD
- U1 pad 6: Net-(R19-Pad1) -> Net-(R21-Pad1)
Routing:
- net +5V: track 19.1 -> 135.6 mm, vias 2 -> 0
- net Net-(R22-Pad1): track 0.00 -> 44.0 mm, vias 0 -> 2
- net Net-(R21-Pad1): track 0.00 -> 34.8 mm, vias 0 -> 2
- net DAC: track 0.00 -> 34.6 mm, vias 0 -> 2
- net VDD: track 0.00 -> 17.3 mm, vias 0 -> 3
- net Net-(JP2-Pad1): track 0.00 -> 8.66 mm, vias 0 -> 2
- net Net-(R18-Pad1): track 26.8 -> 33.0 mm
- net OUT16: track 0.00 -> 6.19 mm
- net OUT17: track 0.00 -> 6.17 mm
- net Net-(R19-Pad1): track 27.4 -> 33.1 mm, vias 2 -> 0
- net vCommon: track 0.00 -> 5.72 mm
- net Net-(R24-Pad1): track 0.00 -> 3.20 mm
- net V24.cts: track 24.5 -> 22.0 mm
- net GND: track 10.5 -> 8.33 mm, vias 3 -> 10
- net DI: track 6.27 -> 5.51 mm
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- added copper zone on F.Cu, net VDD
- removed copper zone on F.Cu, net +5V
Other:
- board size 59.9 x 21.6 mm -> 79.4 x 21.6 mm
- board text added: "17"
- board text added: "18"
- board text added: "E10.1"
- board text added: "common"
- board text added: "var|5V"
- board text removed: "+|-"
- board text removed: "Data"
- board text removed: "E10.0"

Commit message: initial
Parts:
- removed R21, R22: 220, Resistor_SMD:R_0603_1608Metric
- J8: value LED 16-17 -> LED Common
Connections:
- J8 pad 1: OUT17 -> vCommon
- J8 pad 2: OUT16 -> vCommon
- U1 pad 25: Net-(R22-Pad1) -> (no net)
- U1 pad 6: Net-(R21-Pad1) -> (no net)
Routing:
- net vCommon: track 5.72 -> 62.4 mm
- net Net-(R22-Pad1): track 44.0 -> 0.00 mm, vias 2 -> 0
- net Net-(R21-Pad1): track 34.8 -> 0.00 mm, vias 2 -> 0
- net OUT16: track 6.19 -> 0.00 mm
- net OUT17: track 6.17 -> 0.00 mm
Other:
- board text added: "E10.2"
- board text removed: "17"
- board text removed: "18"
- board text removed: "E10.1"
