File: E10.kicad_pcb (KiCad board)
At the start: 2 copper layers, 79.4 x 21.6 mm, 45 parts, among them J1 LED 8-15, J2 WS-bus output, J3 WS-bus input, J4 UPDI, J5 Debug, J6 LED common, J7 LED 0-7, J8 LED Common, U1 AVR-64da32, U2 MIC5205-5.0YM5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

Commit message: Initial commit
Other:
- rule pad_to_mask_clearance: 0.051 -> 0
